Commit message: added possibility to remove wheels

File: src/kmr_description/urdf/kmp200/kmp200_copy.xacro (robot description, xacro)
@@ -13,87 +13,89 @@
   <xacro:property name="track_gauge" value="0.365" />
   <xacro:property name="wheel_base" value="0.56" />
-  <xacro:property name="ground_clearance" value="0.025" /> <!-- distance from wheel-floor contact point to base bottom side-->
-  <xacro:macro name="kmp200" params="robot_name without_wheels:=false">
+  <xacro:property name="ground_clearance" value="0.025" />
+  <!-- distance from wheel-floor contact point to base bottom side-->
+  <xacro:macro name="kmp200" params="robot_name with_wheels:=true">
     <link name="${robot_name}_base_footprint"/>
     <joint name="${robot_name}_footprint_to_base_link" type="fixed">
-        <parent link="${robot_name}_base_footprint"/>
-        <child link="${robot_name}_base_link"/>
-        <origin rpy="0 0 0.0" xyz="0 0 ${ground_clearance}"/>
+      <parent link="${robot_name}_base_footprint"/>
+      <child link="${robot_name}_base_link"/>
+      <origin rpy="0 0 0.0" xyz="0 0 ${ground_clearance}"/>
     </joint>
     <link name="${robot_name}_base_link">
-    	<origin rpy="0 0 0" xyz="0 0 0"/>
-        <visual>
-          <geometry>
-            <mesh filename="package://kmr_description/meshes/kmp200/KMP200.dae"/>
-          </geometry>
-          <material name="White"/>
-        </visual>
-        <collision>
-          <geometry>
-            <mesh filename="package://kmr_description/meshes/kmp200/KMP200.dae"/>
-          </geometry>
-        </collision>
-        <inertial>
-            <origin xyz="0 0 ${center_of_gravity_height_noload-ground_clearance}" rpy="0 0 0"/>
-            <mass value="${base_mass}"/>
-            <!-- obtained from KMP200 model on fusion 360 with some modification to align center of mass with the given one-->
-            <inertia ixx="28.95" ixy="0.0" ixz="0.0" iyy="44.03" iyz="0.0" izz="33.83"/>
-        </inertial>
+      <origin rpy="0 0 0" xyz="0 0 0"/>
+      <visual>
+        <geometry>
+          <mesh filename="package://kmr_description/meshes/kmp200/KMP200.dae"/>
+        </geometry>
+        <material name="White"/>
+      </visual>
+      <collision>
+        <geometry>
+          <mesh filename="package://kmr_description/meshes/kmp200/KMP200.dae"/>
+        </geometry>
+      </collision>
+      <inertial>
+        <origin xyz="0 0 ${center_of_gravity_height_noload-ground_clearance}" rpy="0 0 0"/>
+        <mass value="${base_mass}"/>
+        <!-- obtained from KMP200 model on fusion 360 with some modification to align center of mass with the given one-->
+        <inertia ixx="28.95" ixy="0.0" ixz="0.0" iyy="44.03" iyz="0.0" izz="33.83"/>
+      </inertial>
     </link>
     <joint name="${robot_name}_base_link_to_top" type="fixed">
-        <parent link="${robot_name}_base_link"/>
-        <child link="${robot_name}_base_top_link"/>
-        <origin rpy="0 0 0.0" xyz="0 0 ${base_height-ground_clearance}"/>
+      <parent link="${robot_name}_base_link"/>
+      <child link="${robot_name}_base_top_link"/>
+      <origin rpy="0 0 0.0" xyz="0 0 ${base_height-ground_clearance}"/>
     </joint>
     <link name="${robot_name}_base_top_link"/>
     <joint name="${robot_name}_laser_B1_joint" type="fixed">
-            <parent link="${robot_name}_base_link" />
-            <child link="${robot_name}_laser_B1_link" />
-            <origin xyz="0.464 -0.256 0.1168" rpy="0 0 -0.7854"/>
+      <parent link="${robot_name}_base_link" />
+      <child link="${robot_name}_laser_B1_link" />
+      <origin xyz="0.464 -0.256 0.1168" rpy="0 0 -0.7854"/>
     </joint>
     <link name="${robot_name}_laser_B1_link">
-        <visual>
-          <origin xyz="0 0 0" rpy="3.1413 0 0"/>
-          <geometry>
-              <mesh filename="package://kmr_description/meshes/kmp200/sensors/visual/sick_lms1xx.dae" />
-          </geometry>
-          <material name="DarkGrey"/>
-        </visual>
-        <collision>
-            <origin xyz="0.0 0 0.0" rpy="0 0 0"/>
-            <geometry>
-                <mesh filename="package://kmr_description/meshes/kmp200/sensors/collision/sick_lms1xx.stl" />
-            </geometry>
-        </collision>
-        <inertial>
-            <mass value="1.2"/>
-            <inertia ixx="0.002355" ixy="0.0" ixz="0.0" iyy="0.002355" iyz="0.0" izz="0.0002809"/>
-        </inertial>
+      <visual>
+        <origin xyz="0 0 0" rpy="3.1413 0 0"/>
+        <geometry>
+          <mesh filename="package://kmr_description/meshes/kmp200/sensors/visual/sick_lms1xx.dae" />
+        </geometry>
+        <material name="DarkGrey"/>
+      </visual>
+      <collision>
+        <origin xyz="0.0 0 0.0" rpy="0 0 0"/>
+        <geometry>
+          <mesh filename="package://kmr_description/meshes/kmp200/sensors/collision/sick_lms1xx.stl" />
+        </geometry>
+      </collision>
+      <inertial>
+        <mass value="1.2"/>
+        <inertia ixx="0.002355" ixy="0.0" ixz="0.0" iyy="0.002355" iyz="0.0" izz="0.0002809"/>
+      </inertial>
     </link>
     <joint name="${robot_name}_laser_B4_joint" type="fixed">
-            <parent link="${robot_name}_base_link" />
-            <child link="${robot_name}_laser_B4_link" />
-            <origin xyz="-0.464 0.256 0.1168" rpy="0 0 2.3562"/>
+      <parent link="${robot_name}_base_link" />
+      <child link="${robot_name}_laser_B4_link" />
+      <origin xyz="-0.464 0.256 0.1168" rpy="0 0 2.3562"/>
     </joint>
     <link name="${robot_name}_laser_B4_link">
-        <visual>
-          <origin xyz="0.0 0 0" rpy="0 3.1413 3.1413"/>
-          <geometry>
-              <mesh filename="package://kmr_description/meshes/kmp200/sensors/visual/sick_lms1xx.dae" />
-          </geometry>
-          <material name="DarkGrey"/>
-        </visual>
-        <collision>
-            <origin xyz="0 0 0" rpy="0 0 0"/>
-            <geometry>
-                  <mesh filename="package://kmr_description/meshes/kmp200/sensors/collision/sick_lms1xx.stl" />
-            </geometry>
-        </collision>
-        <inertial>
-            <mass value="1.2"/>
-            <inertia ixx="0.002355" ixy="0.0" ixz="0.0" iyy="0.002355" iyz="0.0" izz="0.0002809"/>
-        </inertial>
+      <visual>
+        <origin xyz="0.0 0 0" rpy="0 3.1413 3.1413"/>
+        <geometry>
+          <mesh filename="package://kmr_description/meshes/kmp200/sensors/visual/sick_lms1xx.dae" />
+        </geometry>
+        <material name="DarkGrey"/>
+      </visual>
+      <collision>
+        <origin xyz="0 0 0" rpy="0 0 0"/>
+        <geometry>
+          <mesh filename="package://kmr_description/meshes/kmp200/sensors/collision/sick_lms1xx.stl" />
+        </geometry>
+      </collision>
+      <inertial>
+        <mass value="1.2"/>
+        <inertia ixx="0.002355" ixy="0.0" ixz="0.0" iyy="0.002355" iyz="0.0" izz="0.0002809"/>
+      </inertial>
     </link>
-    <link name="${robot_name}_front_left_wheel_link">
+    <xacro:if value="${with_wheels}">
+      <link name="${robot_name}_front_left_wheel_link">
         <visual>
           <origin xyz="0 0 0" rpy="0 0 0" />
@@ -108,6 +110,6 @@
           </geometry>
         </collision>
-    </link>
-    <link name="${robot_name}_front_right_wheel_link">
+      </link>
+      <link name="${robot_name}_front_right_wheel_link">
         <visual>
           <origin xyz="0 0 0" rpy="0 0 0" />
@@ -122,6 +124,6 @@
           </geometry>
         </collision>
-    </link>
-    <link name="${robot_name}_back_left_wheel_link">
+      </link>
+      <link name="${robot_name}_back_left_wheel_link">
         <visual>
           <origin xyz="0 0 0" rpy="0 0 0" />
@@ -136,6 +138,6 @@
           </geometry>
         </collision>
-    </link>
-    <link name="${robot_name}_back_right_wheel_link">
+      </link>
+      <link name="${robot_name}_back_right_wheel_link">
         <visual>
           <origin xyz="0 0 0" rpy="0 0 0" />
@@ -154,6 +156,6 @@
             <inertia ixx="0.075016" ixy="0.0" ixz="0.0" iyy="0.075016" iyz="0.0" izz="0.109375"/>
         </inertial> -->
-    </link>
-    <joint name="${robot_name}_front_left_wheel_joint" type="continuous">
+      </link>
+      <joint name="${robot_name}_front_left_wheel_joint" type="continuous">
         <parent link="${robot_name}_base_link"/>
         <child link="${robot_name}_front_left_wheel_link"/>
@@ -162,6 +164,6 @@
         <limit effort="100" velocity="100"/>
         <joint_properties damping="0.0" friction="0.0"/>
-    </joint>
-    <joint name="${robot_name}_front_right_wheel_joint" type="continuous">
+      </joint>
+      <joint name="${robot_name}_front_right_wheel_joint" type="continuous">
         <parent link="${robot_name}_base_link"/>
         <child link="${robot_name}_front_right_wheel_link"/>
@@ -170,6 +172,6 @@
         <limit effort="100" velocity="100"/>
         <joint_properties damping="0.0" friction="0.0"/>
-    </joint>
-    <joint name="${robot_name}_back_left_wheel_joint" type="continuous">
+      </joint>
+      <joint name="${robot_name}_back_left_wheel_joint" type="continuous">
         <parent link="${robot_name}_base_link"/>
         <child link="${robot_name}_back_left_wheel_link"/>
@@ -178,6 +180,6 @@
         <limit effort="100" velocity="100"/>
         <joint_properties damping="0.0" friction="0.0"/>
-    </joint>
-    <joint name="${robot_name}_back_right_wheel_joint" type="continuous">
+      </joint>
+      <joint name="${robot_name}_back_right_wheel_joint" type="continuous">
         <parent link="${robot_name}_base_link"/>
         <child link="${robot_name}_back_right_wheel_link"/>
@@ -186,7 +188,8 @@
         <limit effort="100" velocity="100"/>
         <joint_properties damping="0.0" friction="0.0"/>
-    </joint>
+      </joint>
+    </xacro:if>
     <!--Extensions -->
     <xacro:kmp200_gazebo robot_name="${robot_name}"/>
-   </xacro:macro>
+  </xacro:macro>
 </robot>

File: src/kmr_description/urdf/robot/kmriiwa_copy.urdf.xacro (robot description, xacro)
@@ -4,5 +4,5 @@
   <xacro:include filename="$(find kmr_description)/urdf/iiwa14/materials.xacro" />
   <xacro:include filename="$(find kmr_description)/urdf/iiwa14/iiwa14.xacro"/>
-  <xacro:include filename="$(find kmr_description)/urdf/kmp200/kmp200.xacro"/>
+  <xacro:include filename="$(find kmr_description)/urdf/kmp200/kmp200_copy.xacro"/>
   <xacro:include filename="$(find kmr_description)/urdf/d435/_d435.urdf.xacro"/>
   <xacro:include filename="$(find kmr_description)/urdf/adapters/camera_adapter.urdf.xacro"/>
@@ -23,5 +23,5 @@
   <xacro:arg name="gripper" default="$(find kmr_description)/urdf/gripper/robotiq_gripper.urdf.xacro" />
   <!--kmp200-->
-  <xacro:kmp200 robot_name="$(arg robot_name)"/>
+  <xacro:kmp200 robot_name="$(arg robot_name)" with_wheels="true"/>
   <!--riser flange-->
   <joint name="$(arg robot_name)_base_top_riser_flange_joint" type="fixed">
