Commit message: Fixed closed loop articulation

File: src/kmr_description/urdf/robot/kmriiwa.urdf (robot description, URDF)
Before this commit: robot kmriiwa, 72 links, 72 joints
Joints:
- removed joint joint_adapter_gripper
- joint camera_front_joint: origin xyz=0.5 0 0 rpy=0 0 0 -> xyz=0.5 0 -0.0075 rpy=0 0 0
- joint camera_left_joint: origin xyz=0 0 0 rpy=0 0 1.5707963267948966 -> xyz=0 0 0.005 rpy=0 0 1.5707963267948966
- joint camera_manipulator_joint: origin xyz=0 0.03 0 rpy=0 -1.5707963267948966 -1.5707963267948966 -> xyz=0 0.035 0 rpy=0 -1.5707963267948966 -1.5707963267948966
- joint camera_right_joint: origin xyz=0 0 0 rpy=0 0 -1.5707963267948966 -> xyz=0 0 0.005 rpy=0 0 -1.5707963267948966
- joint left_camera_adapter_joint: origin xyz=0 0.275 0.0125 rpy=0 0 0 -> xyz=0 0.275 0 rpy=0 0 0
- joint right_camera_adapter_joint: origin xyz=0 -0.275 0.0125 rpy=0 0 0 -> xyz=0 -0.275 0 rpy=0 0 0

File: src/kmr_description/urdf/robot/kmriiwa.urdf.xacro (robot description, xacro)
@@ -54,11 +54,11 @@
     <origin xyz="0 0 0.005" rpy="0 0 0" />
   </xacro:gripper>
-  <!-- THese values has to be tuned to match the pysical robot -->
   <!-- Cameras with adapters -->
+  <!-- These values has to be tuned to match the pysical robot -->
   <xacro:camera_adapter parent="$(arg robot_name)_base_top_link" camera_position="left">
     <origin xyz="0 0.275 0" rpy="0 0 0"/>
   </xacro:camera_adapter>
   <xacro:camera_adapter parent="$(arg robot_name)_base_top_link" camera_position="right">
-    <origin xyz="0 -0.275 0.05" rpy="0 0 0"/>
+    <origin xyz="0 -0.275 0" rpy="0 0 0"/>
   </xacro:camera_adapter>
   <xacro:sensor_d435 parent="left_camera_adapter" name="camera_left" use_nominal_extrinsics="true">
