Commit message: created new main kmr.urdf

File: src/kmr_description/urdf/robot/kmr.urdf (robot description, URDF)
Before this commit: robot kmriiwa, 72 links, 71 joints
Links:
- removed link kmriiwa_back_left_wheel_link
- removed link kmriiwa_back_right_wheel_link
- removed link kmriiwa_base_footprint
- removed link kmriiwa_base_link
- removed link kmriiwa_base_top_link
- removed link kmriiwa_front_left_wheel_link
- removed link kmriiwa_front_right_wheel_link
- removed link kmriiwa_laser_B1_link
- removed link kmriiwa_laser_B4_link
- removed link kmriiwa_link_0
- removed link kmriiwa_link_1
- removed link kmriiwa_link_2
- removed link kmriiwa_link_3
- removed link kmriiwa_link_4
- removed link kmriiwa_link_5
- removed link kmriiwa_link_6
- removed link kmriiwa_link_7
- removed link kmriiwa_link_ee
- removed link kmriiwa_riser_flange_link
- removed link left_inner_finger
- removed link left_inner_knuckle
- removed link left_outer_finger
- removed link left_outer_knuckle
- removed link right_inner_finger
- removed link right_inner_knuckle
- removed link right_outer_finger
- removed link right_outer_knuckle
- added link gripper_left_inner_finger, mass 0.00724255346165745; collision mesh filename=package://kmr_description/meshes/gripper/inner_finger_coars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; visual mesh filename=package://kmr_description/meshes/gripper/inner_finger_fine.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
- added link gripper_left_inner_knuckle, mass 0.0110930853895903; collision mesh filename=package://kmr_description/meshes/gripper/inner_knuckle_coar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; visual mesh filename=package://kmr_description/meshes/gripper/inner_knuckle_fine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
- added link gripper_left_outer_finger, mass 0.0273093985570947; collision mesh filename=package://kmr_description/meshes/gripper/outer_finger_coars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; visual mesh filename=package://kmr_description/meshes/gripper/outer_finger_fine.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
- added link gripper_left_outer_knuckle, mass 0.00684838849434396; collision mesh filename=package://kmr_description/meshes/gripper/outer_knuckle_coar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; visual mesh filename=package://kmr_description/meshes/gripper/outer_knuckle_fine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
- added link gripper_right_inner_finger, mass 0.00724255346165744; collision mesh filename=package://kmr_description/meshes/gripper/inner_finger_coars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; visual mesh filename=package://kmr_description/meshes/gripper/inner_finger_fine.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
- added link gripper_right_inner_knuckle, mass 0.0110930853895903; collision mesh filename=package://kmr_description/meshes/gripper/inner_knuckle_coar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; visual mesh filename=package://kmr_description/meshes/gripper/inner_knuckle_fine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
- added link gripper_right_outer_finger, mass 0.0273093985570947; collision mesh filename=package://kmr_description/meshes/gripper/outer_finger_coars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; visual mesh filename=package://kmr_description/meshes/gripper/outer_finger_fine.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
- added link gripper_right_outer_knuckle, mass 0.00684838849401352; collision mesh filename=package://kmr_description/meshes/gripper/outer_knuckle_coar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; visual mesh filename=package://kmr_description/meshes/gripper/outer_knuckle_fine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
- added link kmr_back_left_wheel_link; collision cylinder length=0.132 radius=0.125; visual mesh filename=package://kmr_description/meshes/kmp200/wheels/omni_wheel_1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 scale=1.06695 1.06695 1.06695
- added link kmr_back_right_wheel_link; collision cylinder length=0.132 radius=0.125; visual mesh filename=package://kmr_description/meshes/kmp200/wheels/omni_wheel_1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 scale=1.06695 1.06695 1.06695
- added link kmr_base_footprint
- added link kmr_base_link, mass 390; collision mesh filename=package://kmr_description/meshes/kmp200/KMP200.dae; visual mesh filename=package://kmr_description/meshes/kmp200/KMP200.dae
- added link kmr_base_top_link
- added link kmr_front_left_wheel_link; collision cylinder length=0.132 radius=0.125; visual mesh filename=package://kmr_description/meshes/kmp200/wheels/omni_wheel_1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 scale=1.06695 1.06695 1.06695
- added link kmr_front_right_wheel_link; collision cylinder length=0.132 radius=0.125; visual mesh filename=package://kmr_description/meshes/kmp200/wheels/omni_wheel_1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 scale=1.06695 1.06695 1.06695
- added link kmr_laser_B1_link, mass 1.2; collision mesh filename=package://kmr_description/meshes/kmp200/sensors/collision/s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; visual mesh filename=package://kmr_description/meshes/kmp200/sensors/visual/sick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
- added link kmr_laser_B4_link, mass 1.2; collision mesh filename=package://kmr_description/meshes/kmp200/sensors/collision/s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; visual mesh filename=package://kmr_description/meshes/kmp200/sensors/visual/sick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
- added link kmr_link_0, mass 5; collision mesh filename=package://kmr_description/meshes/iiwa14/collision/link_0.stl; visual mesh filename=package://kmr_description/meshes/iiwa14/visual/link_0.stl
- added link kmr_link_1, mass 4; collision mesh filename=package://kmr_description/meshes/iiwa14/collision/link_1.stl; visual mesh filename=package://kmr_description/meshes/iiwa14/visual/link_1.stl
- added link kmr_link_2, mass 4; collision mesh filename=package://kmr_description/meshes/iiwa14/collision/link_2.stl; visual mesh filename=package://kmr_description/meshes/iiwa14/visual/link_2.stl
- added link kmr_link_3, mass 3; collision mesh filename=package://kmr_description/meshes/iiwa14/collision/link_3.stl; visual mesh filename=package://kmr_description/meshes/iiwa14/visual/link_3.stl
- added link kmr_link_4, mass 2.7; collision mesh filename=package://kmr_description/meshes/iiwa14/collision/link_4.stl; visual mesh filename=package://kmr_description/meshes/iiwa14/visual/link_4.stl
- added link kmr_link_5, mass 1.7; collision mesh filename=package://kmr_description/meshes/iiwa14/collision/link_5.stl; visual mesh filename=package://kmr_description/meshes/iiwa14/visual/link_5.stl
- added link kmr_link_6, mass 1.8; collision mesh filename=package://kmr_description/meshes/iiwa14/collision/link_6.stl; visual mesh filename=package://kmr_description/meshes/iiwa14/visual/link_6.stl
- added link kmr_link_7, mass 0.3; collision mesh filename=package://kmr_description/meshes/iiwa14/collision/link_7.stl; visual mesh filename=package://kmr_description/meshes/iiwa14/visual/link_7.stl
- added link kmr_link_ee
- added link kmr_riser_flange_link; collision cylinder length=0.0 radius=0.121; visual cylinder length=0.0 radius=0.121
Joints:
- removed joint finger_joint
- removed joint iiwa14_joint_gripper
- removed joint kmriiwa_back_left_wheel_joint
- removed joint kmriiwa_back_right_wheel_joint
- removed joint kmriiwa_base_link_to_top
- removed joint kmriiwa_base_top_riser_flange_joint
- removed joint kmriiwa_footprint_to_base_link
- removed joint kmriiwa_front_left_wheel_joint
- removed joint kmriiwa_front_right_wheel_joint
- removed joint kmriiwa_joint_1
- removed joint kmriiwa_joint_2
- removed joint kmriiwa_joint_3
- removed joint kmriiwa_joint_4
- removed joint kmriiwa_joint_5
- removed joint kmriiwa_joint_6
- removed joint kmriiwa_joint_7
- removed joint kmriiwa_joint_ee
- removed joint kmriiwa_laser_B1_joint
- removed joint kmriiwa_laser_B4_joint
- removed joint kmriiwa_riser_flange_link_kmriiwa_joint
- removed joint left_inner_finger_joint
- removed joint left_inner_knuckle_joint
- removed joint left_outer_finger_joint
- removed joint right_inner_finger_joint
- removed joint right_inner_knuckle_joint
- removed joint right_outer_finger_joint
- removed joint right_outer_knuckle_joint
- added joint gripper_adapter_joint_gripper: type fixed, parent gripper_adapter, child gripper_base_link, origin xyz=0 0 0.005 rpy=0 0 0
- added joint gripper_finger_joint: type revolute, parent gripper_base_link, child gripper_left_outer_knuckle, origin xyz=0.0306011444260539 0 0.0627920162695395 rpy=0 0 0, axis 0 -1 0, limit lower=0 upper=0.725 effort=1000 velocity=2.0
- added joint gripper_left_inner_finger_joint: type revolute, parent gripper_left_inner_knuckle, child gripper_left_inner_finger, origin xyz=0.034585310861294 0 0.0454970193817975 rpy=0 0 0, axis 0 -1 0, limit lower=0 upper=0.8757 effort=1000 velocity=2.0, mimic joint=gripper_finger_joint multiplier=-1 offset=0
- added joint gripper_left_inner_knuckle_joint: type revolute, parent gripper_base_link, child gripper_left_inner_knuckle, origin xyz=0.0127000000001501 0 0.0693074999999639 rpy=0 0 0, axis 0 -1 0, limit lower=0 upper=0.8757 effort=1000 velocity=2.0, mimic joint=gripper_finger_joint multiplier=1 offset=0
- added joint gripper_left_outer_finger_joint: type fixed, parent gripper_left_outer_knuckle, child gripper_left_outer_finger, origin xyz=0.0316910442266543 0 -0.00193396375724605 rpy=0 0 0, axis 0 -1 0
- added joint gripper_right_inner_finger_joint: type revolute, parent gripper_right_inner_knuckle, child gripper_right_inner_finger, origin xyz=0.0341060475457406 0 0.0458573878541688 rpy=0 0 0, axis 0 1 0, limit lower=0 upper=0.8757 effort=1000 velocity=2.0, mimic joint=gripper_finger_joint multiplier=1 offset=0
- added joint gripper_right_inner_knuckle_joint: type revolute, parent gripper_base_link, child gripper_right_inner_knuckle, origin xyz=-0.0126999999998499 0 0.0693075000000361 rpy=0 0 3.14159265358979, axis 0 1 0, limit lower=0 upper=0.8757 effort=1000 velocity=2.0, mimic joint=gripper_finger_joint multiplier=-1 offset=0
- added joint gripper_right_outer_finger_joint: type fixed, parent gripper_right_outer_knuckle, child gripper_right_outer_finger, origin xyz=0.0317095909367246 0 -0.0016013564954687 rpy=0 0 0, axis 0 1 0
- added joint gripper_right_outer_knuckle_joint: type revolute, parent gripper_base_link, child gripper_right_outer_knuckle, origin xyz=-0.0306011444258893 0 0.0627920162695395 rpy=0 0 3.14159265358979, axis 0 1 0, limit lower=0 upper=0.8757 effort=1000 velocity=2.0, mimic joint=gripper_finger_joint multiplier=-1 offset=0
- added joint kmr_back_left_wheel_joint: type continuous, parent kmr_base_link, child kmr_back_left_wheel_link, origin xyz=-0.28 0.1825 0.1, axis 0 1 0, limit effort=100 velocity=100
- added joint kmr_back_right_wheel_joint: type continuous, parent kmr_base_link, child kmr_back_right_wheel_link, origin xyz=-0.28 -0.1825 0.1, axis 0 1 0, limit effort=100 velocity=100
- added joint kmr_base_link_to_top: type fixed, parent kmr_base_link, child kmr_base_top_link, origin xyz=0 0 0.6749999999999999 rpy=0 0 0.0
- added joint kmr_base_top_riser_flange_joint: type fixed, parent kmr_base_top_link, child kmr_riser_flange_link, origin xyz=0.363 -0.184 -0.01 rpy=0 0 -1.5708
- added joint kmr_footprint_to_base_link: type fixed, parent kmr_base_footprint, child kmr_base_link, origin xyz=0 0 0.025 rpy=0 0 0.0
- added joint kmr_front_left_wheel_joint: type continuous, parent kmr_base_link, child kmr_front_left_wheel_link, origin xyz=0.28 0.1825 0.1, axis 0 1 0, limit effort=100 velocity=100
- added joint kmr_front_right_wheel_joint: type continuous, parent kmr_base_link, child kmr_front_right_wheel_link, origin xyz=0.28 -0.1825 0.1, axis 0 1 0, limit effort=100 velocity=100
- added joint kmr_joint_1: type revolute, parent kmr_link_0, child kmr_link_1, origin xyz=0 0 0.1575 rpy=0 0 0, axis 0 0 1, limit lower=-2.9670597283903604 upper=2.9670597283903604 effort=300 velocity=10
- added joint kmr_joint_2: type revolute, parent kmr_link_1, child kmr_link_2, origin xyz=0 0 0.2025 rpy=1.5707963267948966   0 3.141592653589793, axis 0 0 1, limit lower=-2.0943951023931953 upper=2.0943951023931953 effort=300 velocity=10
- added joint kmr_joint_3: type revolute, parent kmr_link_2, child kmr_link_3, origin xyz=0 0.2045 0 rpy=1.5707963267948966 0 3.141592653589793, axis 0 0 1, limit lower=-2.9670597283903604 upper=2.9670597283903604 effort=300 velocity=10
- added joint kmr_joint_4: type revolute, parent kmr_link_3, child kmr_link_4, origin xyz=0 0 0.2155 rpy=1.5707963267948966 0 0, axis 0 0 1, limit lower=-2.0943951023931953 upper=2.0943951023931953 effort=300 velocity=10
- added joint kmr_joint_5: type revolute, parent kmr_link_4, child kmr_link_5, origin xyz=0 0.1845 0 rpy=-1.5707963267948966 3.141592653589793 0, axis 0 0 1, limit lower=-2.9670597283903604 upper=2.9670597283903604 effort=300 velocity=10
- added joint kmr_joint_6: type revolute, parent kmr_link_5, child kmr_link_6, origin xyz=0 0 0.2155 rpy=1.5707963267948966 0 0, axis 0 0 1, limit lower=-2.0943951023931953 upper=2.0943951023931953 effort=300 velocity=10
- added joint kmr_joint_7: type revolute, parent kmr_link_6, child kmr_link_7, origin xyz=0 0.081 0 rpy=-1.5707963267948966 3.141592653589793 0, axis 0 0 1, limit lower=-3.0543261909900763 upper=3.0543261909900763 effort=300 velocity=10
- added joint kmr_joint_ee: type fixed, parent kmr_link_7, child kmr_link_ee, origin xyz=0 0 0.045 rpy=0 0 0
- added joint kmr_laser_B1_joint: type fixed, parent kmr_base_link, child kmr_laser_B1_link, origin xyz=0.464 -0.256 0.1168 rpy=0 0 -0.7854
- added joint kmr_laser_B4_joint: type fixed, parent kmr_base_link, child kmr_laser_B4_link, origin xyz=-0.464 0.256 0.1168 rpy=0 0 2.3562
- added joint kmr_riser_flange_link_kmr_joint: type fixed, parent kmr_riser_flange_link, child kmr_link_0, origin xyz=0 0 0.0 rpy=0 0 0
- joint camera_front_joint: parent kmriiwa_base_top_link -> kmr_base_top_link
- joint joint_a7_adapter: parent kmriiwa_link_ee -> kmr_link_ee
- joint left_camera_adapter_joint: parent kmriiwa_base_top_link -> kmr_base_top_link
- joint right_camera_adapter_joint: parent kmriiwa_base_top_link -> kmr_base_top_link
